File: Amplifier/Amplifier.kicad_sch (KiCad schematic)
At the start: 14 parts, among them J1 Conn_01x01_Pin, J2 Conn_01x01_Pin, J3 Conn_01x01_Pin, J4 Conn_01x01_Pin, J5 Conn_01x01_Pin, J6 Conn_01x01_Pin, J7 Conn_01x01_Pin, Q1 BC557, Q2 BD138

Commit message: ...
Parts:
- C1: value C -> 100n
- Q2: value BD138 -> BD179
- R1: value R -> 2k2
- R2, R3: value R -> 100
Connections:
- net at J4.1 (Pin_1): now also C1.1, D1.1 (K), J6.1 (Pin_1)
- net at Q2.1 (E): now also J3.1 (Pin_1), J7.1 (Pin_1)
- net at D1.2 (A), Q2.2 (C), R3.2: now also J5.1 (Pin_1)
Other:
- moved on the sheet: C1, D1, J1, J2, J4, J7, R3
