File: AVR/AVR.kicad_sch (KiCad schematic)
At the start: 1 part, among them U1 ATmega88-20P

Commit message: ...
Parts:
- added 5V&GND: Conn_01x02_Pin, Connector_PinHeader_2.00mm:PinHeader_1x02_P2.00mm_Vertical, symbol Connector:Conn_01x02_Pin
- added ADC_Input: Conn_01x01_Pin, Connector_PinHeader_1.00mm:PinHeader_1x01_P1.00mm_Vertical, symbol Connector:Conn_01x01_Pin
- added C1, C2, C3: 100nF, Capacitor_THT:C_Disc_D3.0mm_W2.0mm_P2.50mm, symbol Device:C
- added D1: RED, symbol Device:LED
- added D2, D3, D4, D5: LED, symbol Device:LED
- added D6: D_Zener, symbol Device:D_Zener
- added Encoder, TX/RX_Interface: Conn_01x04_Pin, Connector_PinHeader_1.00mm:PinHeader_1x04_P1.00mm_Vertical, symbol Connector:Conn_01x04_Pin
- added PWM&5V: Conn_01x02_Pin, Connector_PinHeader_1.00mm:PinHeader_1x02_P1.00mm_Vertical, symbol Connector:Conn_01x02_Pin
- added R1: 4.7k, symbol Device:R
- added R2: 330, symbol Device:R
- added R3, R4, R5, R6: R, symbol Device:R
- added SPI: Conn_01x06_Pin, Connector_PinHeader_1.00mm:PinHeader_2x03_P1.00mm_Vertical, symbol Connector:Conn_01x06_Pin
Connections:
- net at U1.1 (~{RESET}/PC6): now also C3.1, D6.2 (A), R1.2, SPI.RST (Pin_5)
- net at U1.15 (PB1): now also PWM&5V.PWM (Pin_2), R3.1
- net at U1.17 (PB3): now also SPI.MOSI (Pin_4)
- net at U1.18 (PB4): now also SPI.MISO (Pin_1)
- net at U1.19 (PB5): now also SPI.SCK (Pin_3)
- net at U1.2 (PD0): now also TX/RX_Interface.TX (Pin_2)
- net at U1.20 (AVCC): now also U1.21 (AREF), U1.7 (VCC), 5V&GND.5V (Pin_1), C1.1, C2.1, D6.1 (K), Encoder.5V (Pin_1), PWM&5V.5V (Pin_1), R1.1, R2.1, SPI.VTG (Pin_2), TX/RX_Interface.5V (Pin_3)
- net at U1.22 (GND), U1.8 (GND): now also 5V&GND.GND (Pin_2), C1.2, C2.2, C3.2, D1.1 (K), D2.1 (K), Encoder.GND (Pin_4), SPI.GND (Pin_6), TX/RX_Interface.GND (Pin_4)
- net at U1.23 (PC0): now also Encoder.D1 (Pin_2)
- net at U1.24 (PC1): now also Encoder.D2 (Pin_3)
- net at U1.25 (PC2): now also ADC_Input.1 (Pin_1)
- net at U1.3 (PD1): now also TX/RX_Interface.RX (Pin_1)
- new net: D2.2 (A), R3.2
- new net: D1.2 (A), R2.2
Other:
- moved on the sheet: U1
